Commit message: Correct arm origin position

File: src/third-party/mycobot-ros2/mycobot_description/urdf/mech/mycobot_320_arm.urdf.xacro (robot description, xacro)
@@ -149,5 +149,5 @@
       <parent link="${prefix}link1"/>
       <child link="${prefix}link2"/>
-      <origin xyz= "0.0 0.0 0.162" rpy = "0 0 0"/>
+      <origin xyz= "0.0 0.0 0.162" rpy = "0 0 ${pi/2}"/>
       <dynamics damping="${joint_damping}" friction="${joint_friction}"/>
     </joint>
@@ -181,5 +181,5 @@
       <parent link="${prefix}link5"/>
       <child link="${prefix}link6"/>
-      <origin xyz="0 -0.084 0" rpy="${pi/2} 0 0"/>
+      <origin xyz="0 -0.084 0" rpy="${pi/2} ${-pi/2} 0"/>
       <dynamics damping="${joint_damping}" friction="${joint_friction}"/>
     </joint>
